Commit message: fix urdf's bug.

File: urdf/common/swerve_drive.urdf.xacro (robot description, xacro)
@@ -48,8 +48,8 @@
         <joint name="${prefix}_wheel_joint" type="revolute">
             <axis xyz="0 1 0"/>
-            <origin xyz="0 0 -0.06635" rpy="0 0 0"/>
+            <origin xyz="0 0 -0.07735" rpy="0 0 0"/>
             <parent link="${prefix}_pivot"/>
             <child link="${prefix}_wheel"/>
-            <limit effort="3" velocity="76" lower="-1e10" upper="1e10"/>
+            <limit effort="3.0" velocity="100" lower="-1e10" upper="1e10"/>
             <dynamics damping="0.0" friction="0.05"/>
         </joint>

File: urdf/sentry/chassis.urdf.xacro (robot description, xacro)
@@ -42,4 +42,8 @@
         <xacro:swerve_transmission prefix="left_back" wheel_reduction="13" pivot_offset="-0.259"/>   <!-- 6.0335-->
         <xacro:swerve_transmission prefix="right_back" wheel_reduction="13" pivot_offset="2.330"/>   <!-- -3.923-->
+<!--        <xacro:swerve_transmission prefix="left_front" wheel_reduction="13" pivot_offset="0"/>   &lt;!&ndash; 2.3566&ndash;&gt;-->
+<!--        <xacro:swerve_transmission prefix="right_front" wheel_reduction="13" pivot_offset="0"/>   &lt;!&ndash; -0.283&ndash;&gt;-->
+<!--        <xacro:swerve_transmission prefix="left_back" wheel_reduction="13" pivot_offset="0"/>   &lt;!&ndash; 6.0335&ndash;&gt;-->
+<!--        <xacro:swerve_transmission prefix="right_back" wheel_reduction="13" pivot_offset="0"/>   &lt;!&ndash; -3.923&ndash;&gt;-->
     </xacro:macro>
 </robot>
